Commit message: initial pass at making geometries

File: src/models/KR5_ACR_model.urdf (robot description, URDF)
Before this commit: robot kuka_kr5_arc, 9 links, 8 joints
Links:
- link base_link: geometry collision box size=.532 .376 .225
- link link_1: geometry collision box size=.483 .465 .332
- link link_2: geometry collision box size=.751 .208 .472
- link link_3: geometry collision box size=.627 .279 .440
- link link_4: geometry collision box size=.155 .132 .313
- link link_5: geometry collision box size=.157 .097 .101
- link link_6: geometry collision box size=.05 .05 .006
